File: esp32-board-v1.1/esp32-board-v1.1.kicad_sch (KiCad schematic)
At the start: 106 parts, among them J1 USB-C 2.0 Sink, J2 GDEM102T91 24P FPC, J3 MicroSD, J4 BAT1, J5 BAT2, Q1 Si1304BDL, SW1 RESET, SW2 BOOT, SW3 KEY1, SW4 KEY2, SW5 KEY3, U1 ESP32-S3-WROOM-1-N16R8, U2 BQ25895RTW, U3 TPS63070, U4 MAX17048, U5 TUSB320LI, U6 TPS22918

Commit message: 调整pcb布局
Parts:
- J4, J5: footprint Connector_Hirose:Hirose_DF13-02P-1.25DS_1x02_P1.25mm_Horizontal -> Connector_Molex:Molex_PicoBlade_53261-0271_1x02-1MP_P1.25mm_Horizontal; MPN Hirose DF13A-2P-1.25H(21) -> Molex 53261-0271; Status PROVISIONAL -> RELEASED
- U2: MPN BQ25895RTW -> BQ25895RTWT
- U3: MPN TPS63070 -> TPS63070RNMT; Status RELEASED -> PROVISIONAL
- U4: MPN MAX17048 -> MAX17048G+T10
- U5: MPN TUSB320LI -> TUSB320LIRWBR; Status PROVISIONAL -> RELEASED

Commit message: 优化pcb布局
Parts:
- removed J4: BAT1, Connector_Molex:Molex_PicoBlade_53261-0271_1x02-1MP_P1.25mm_Horizontal, symbol Connector_Generic:Conn_01x02
- removed J5: BAT2, Connector_Molex:Molex_PicoBlade_53261-0271_1x02-1MP_P1.25mm_Horizontal, symbol Connector_Generic:Conn_01x02
- removed U3: TPS63070, Package_DFN_QFN:VQFN-16-1EP_3x3mm_P0.5mm_EP1.45x1.45mm_ThermalVias, symbol local:TPS63070
- added J4: BAT1, Connector_Molex:Molex_PicoBlade_53261-0271_1x02-1MP_P1.25mm_Horizontal, symbol local:CONN_01X02_PICO
- added J5: BAT2, Connector_Molex:Molex_PicoBlade_53261-0271_1x02-1MP_P1.25mm_Horizontal, symbol local:CONN_01X02_PICO
- added U3: TPS63070RNMT, esp32-board-v1.1:RNM0015A, symbol local:TPS63070RNM
- J2: footprint Connector_FFC-FPC:Hirose_FH12-24S-0.5SH_1x24-1MP_P0.50mm_Horizontal -> Connector_FFC-FPC:Amphenol_F32Q-1A7x1-11024_1x24-1MP_P0.5mm_Horizontal; MPN 24P 0.5mm Top-Contact low profile -> Amphenol F32Q-1A7x1-11024 (24P 0.5mm TOP contact)
- J3: footprint Connector_Card:microSD_HC_Hirose_DM3AT-SF-PEJM5 -> esp32-board-v1.1:microSD_DM3AT-SF-PEJM5_EPDF
- U1: footprint RF_Module:ESP32-S3-WROOM-1 -> esp32-board-v1.1:ESP32-S3-WROOM-1_EPDF
Connections:
- net 3V3_MAIN: now also U3.7 (VOUT), U3.8 (VOUT)
- net BAT1_RAW: now also J4.1 (Pin_1)
- net BAT2_RAW: now also J5.1 (Pin_1)
- net GND: now also J4.2 (Pin_2), J5.2 (Pin_2), U3.10 (PGND), U3.4 (GND)
- net SYS: now also U3.12 (VIN), U3.13 (VIN)
- net TPS_EN: now also U3.14 (EN)
- net TPS_FB: now also U3.5 (FB)
- net TPS_L1: now also U3.11 (L1)
- net TPS_L2: now also U3.9 (L2)
- net TPS_PG: now also U3.2 (PG)
- net TPS_PS_SYNC: now also U3.1 (PS/SYNC)
- net TPS_VAUX: now also U3.3 (VAUX)
- net TPS_VSEL: now also U3.15 (VSEL)
Other:
- note added: "/CE = CHG_CE (GPIO47), 10k pull-up to 3V3_MAIN -> charge DISABLED at power-up."
- note added: "Bench test at peak load (Wi-Fi TX + EPD refresh + TF card + CPU) required: measure J4/J5 peak current and connector /"
- note added: "Charge policy (V1.3, review list 2.2 / 2.3)"
- note added: "ICHG default = 896 mA (14 x 64 mA) - keeps the Molex 53261-0271 connector, 26 AWG harness and terminals inside their thermal budget."
- note added: "Start-up: MCU boot -> I2C init -> write ICHG / IINLIM / ITERM / VREG -> read back and verify -> drive /CE LOW -> charging enabled."
- note added: "terminal / harness temperature rise; limit concurrent load in firmware if the design target is exceeded."

Commit message: 调整pcb布局
Parts:
- J1, J3, SW1, SW2, SW3, SW4, SW5: Status PROVISIONAL -> RELEASED
- J2: footprint Connector_FFC-FPC:Amphenol_F32Q-1A7x1-11024_1x24-1MP_P0.5mm_Horizontal -> esp32-board-v1.1:X05B20U24T; MPN Amphenol F32Q-1A7x1-11024 (24P 0.5mm TOP contact) -> XKB X05B20U24T; Status PROVISIONAL -> RELEASED
- L2: footprint Inductor_SMD:L_Coilcraft_XAL4030-XXX -> Inductor_SMD:L_Sunlord_MWSA0402S; MPN Coilcraft XAL4030 / Isat>=3A -> Sunlord MWSA0402S-1R2MT; Status PROVISIONAL -> RELEASED
- NTC1: value 10k 103AT -> 10k B3435; MPN 103AT-2 class NTC -> Vishay NTCS0603E3103FLT; Status PROVISIONAL -> RELEASED
- Q1: footprint Package_TO_SOT_SMD:SOT-23 -> Package_TO_SOT_SMD:SOT-323_SC-70; MPN Si1304BDL / Si1308EDL or compatible -> Si1304BDL-T1-GE3; Status PROVISIONAL -> RELEASED

Commit message: 更新bom料号
Parts:
- D1: MPN (none) -> PESD5V0S1BA,115（华秋 G0089294）; Status PROVISIONAL -> RELEASED
- D2, D3: MPN (none) -> GBLC05C（华秋 G5954860）; Status PROVISIONAL -> RELEASED
- D4, D5: MPN (none) -> LESD3Z5.0CMT1G（华秋 G4193578）; Status PROVISIONAL -> RELEASED
- D6, D7, D8: MPN MBR0530 -> MBR0530T1G（华秋 G3325533）; Status PROVISIONAL -> RELEASED
- F1, F2, F3: MPN (none) -> BSMD0805L-200（华秋 G5053245）; Status PROVISIONAL -> RELEASED
- L1: footprint Inductor_SMD:L_Coilcraft_XAL5030-XXX -> Inductor_SMD:L_Sunlord_MWSA0503S; MPN Coilcraft XAL5030 / Isat>=4.5A -> Sunlord MWSA0503S-1R0MT（华秋 G4719678）; Status PROVISIONAL -> RELEASED
- L3: footprint Inductor_SMD:L_Taiyo-Yuden_NR-40xx -> Inductor_SMD:L_Changjiang_FNR4020S; MPN 47uH >=500mA, low profile -> cjiang FHD4020S-470MT（华秋 G6635066）; Status PROVISIONAL -> RELEASED
- R13: MPN (none) -> 0603WAF1800T5E（华秋 G3705022）; Status PROVISIONAL -> RELEASED
Changed lines of the file:
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@@
 			)
 		)
-		(property "Status" "PROVISIONAL"
+		(property "Status" "RELEASED"
+			(at 27.9400 302.2600 0)
+			(hide yes)
+			(effects
+				(font
+					(size 1.27 1.27)
+				)
+			)
+		)
+		(property "MPN" "BSMD0805L-200（华秋 G5053245）"
 			(at 27.9400 302.2600 0)
 			(hide yes)
@@
 			)
 		)
-		(property "Status" "PROVISIONAL"
+		(property "Status" "RELEASED"
+			(at 44.4500 302.2600 0)
+			(hide yes)
+			(effects
+				(font
+					(size 1.27 1.27)
+				)
+			)
+		)
+		(property "MPN" "PESD5V0S1BA,115（华秋 G0089294）"
 			(at 44.4500 302.2600 0)
 			(hide yes)
@@
 			)
 		)
-		(property "Status" "PROVISIONAL"
+		(property "Status" "RELEASED"
+			(at 60.9600 302.2600 0)
+			(hide yes)
+			(effects
+				(font
+					(size 1.27 1.27)
+				)
+			)
+		)
+		(property "MPN" "GBLC05C（华秋 G5954860）"
 			(at 60.9600 302.2600 0)
 			(hide yes)
@@
 			)
 		)
-		(property "Status" "PROVISIONAL"
+		(property "Status" "RELEASED"
+			(at 77.4700 302.2600 0)
+			(hide yes)
+			(effects
+				(font
+					(size 1.27 1.27)
+				)
+			)
+		)
+		(property "MPN" "GBLC05C（华秋 G5954860）"
 			(at 77.4700 302.2600 0)
 			(hide yes)
@@
 			)
 		)
-		(property "Status" "PROVISIONAL"
+		(property "Status" "RELEASED"
+			(at 93.9800 302.2600 0)
+			(hide yes)
+			(effects
+				(font
+					(size 1.27 1.27)
+				)
+			)
+		)
+		(property "MPN" "LESD3Z5.0CMT1G（华秋 G4193578）"
 			(at 93.9800 302.2600 0)
 			(hide yes)
@@
 			)
 		)
-		(property "Status" "PROVISIONAL"
+		(property "Status" "RELEASED"
+			(at 110.4900 302.2600 0)
+			(hide yes)
+			(effects
+				(font
+					(size 1.27 1.27)
+				)
+			)
+		)
+		(property "MPN" "LESD3Z5.0CMT1G（华秋 G4193578）"
 			(at 110.4900 302.2600 0)
 			(hide yes)
@@
 			)
 		)
-		(property "Footprint" "Inductor_SMD:L_Coilcraft_XAL5030-XXX"
+		(property "Footprint" "Inductor_SMD:L_Sunlord_MWSA0503S"
 			(at 351.7900 127.0000 0)
 			(hide yes)
@@
 			)
 		)
-		(property "Status" "PROVISIONAL"
+		(property "Status" "RELEASED"
 			(at 351.7900 127.0000 0)
 			(hide yes)
@@
 			)
 		)
-		(property "MPN" "Coilcraft XAL5030 / Isat>=4.5A"
+		(property "MPN" "Sunlord MWSA0503S-1R0MT（华秋 G4719678）"
 			(at 351.7900 127.0000 0)
 			(hide yes)
@@
 			)
 		)
-		(property "Status" "PROVISIONAL"
+		(property "Status" "RELEASED"
+			(at 236.2200 140.9700 0)
+			(hide yes)
+			(effects
+				(font
+					(size 1.27 1.27)
+				)
+			)
+		)
+		(property "MPN" "0603WAF1800T5E（华秋 G3705022）"
 			(at 236.2200 140.9700 0)
 			(hide yes)
@@
 			)
 		)
-		(property "Status" "PROVISIONAL"
+		(property "Status" "RELEASED"
+			(at 236.2200 251.4600 0)
+			(hide yes)
+			(effects
+				(font
+					(size 1.27 1.27)
+				)
+			)
+		)
+		(property "MPN" "BSMD0805L-200（华秋 G5053245）"
 			(at 236.2200 251.4600 0)
 			(hide yes)
@@
 			)
 		)
-		(property "Status" "PROVISIONAL"
+		(property "Status" "RELEASED"
+			(at 252.7300 251.4600 0)
+			(hide yes)
+			(effects
+				(font
+					(size 1.27 1.27)
+				)
+			)
+		)
+		(property "MPN" "BSMD0805L-200（华秋 G5053245）"
 			(at 252.7300 251.4600 0)
 			(hide yes)
@@
 			)
 		)
-		(property "Footprint" "Inductor_SMD:L_Taiyo-Yuden_NR-40xx"
+		(property "Footprint" "Inductor_SMD:L_Changjiang_FNR4020S"
 			(at 468.6300 280.6700 0)
 			(hide yes)
@@
 			)
 		)
-		(property "Status" "PROVISIONAL"
+		(property "Status" "RELEASED"
 			(at 468.6300 280.6700 0)
 			(hide yes)
@@
 			)
 		)
-		(property "MPN" "47uH >=500mA, low profile"
+		(property "MPN" "cjiang FHD4020S-470MT（华秋 G6635066）"
 			(at 468.6300 280.6700 0)
 			(hide yes)
@@
 			)
 		)
-		(property "Status" "PROVISIONAL"
+		(property "Status" "RELEASED"
 			(at 534.6700 280.6700 0)
 			(hide yes)
@@
 			)
 		)
-		(property "MPN" "MBR0530"
+		(property "MPN" "MBR0530T1G（华秋 G3325533）"
 			(at 534.6700 280.6700 0)
 			(hide yes)
@@
 			)
 		)
-		(property "Status" "PROVISIONAL"
+		(property "Status" "RELEASED"
 			(at 419.1000 294.6400 0)
 			(hide yes)
@@
 			)
 		)
-		(property "MPN" "MBR0530"
+		(property "MPN" "MBR0530T1G（华秋 G3325533）"
 			(at 419.1000 294.6400 0)
 			(hide yes)
@@
 			)
 		)
-		(property "Status" "PROVISIONAL"
+		(property "Status" "RELEASED"
 			(at 435.6100 294.6400 0)
 			(hide yes)
@@
 			)
 		)
-		(property "MPN" "MBR0530"
+		(property "MPN" "MBR0530T1G（华秋 G3325533）"
 			(at 435.6100 294.6400 0)
 			(hide yes)

Commit message: 补充料号修正文档
Parts:
- C1, C13, C14, C21, C22, C23: MPN (none) -> TCC0805X5R226K250FT（华秋 G14559843）; Populate (none) -> FIT
- C10, C11, C17, C24, C26, C3, C38, C4, C5, C6, C7, C8, C9, D1, D2, D3, D4, D5, D6, D7, D8, F1, F2, F3, J1, J2, J3, J4, J5, L1, L2, L3, NTC1, Q1, R1, R10, R11, R12, R13, R14, R15, R18, R19, R2, R20, R22, R25, R26, R27, R28, R29, R3, R30, R31, R32, R33, R34, R35, R36, R4, R5, R6, R7, R8, R9, SW1, SW2, SW3, SW4, SW5, U1, U2, U3, U4, U5, U6: Populate (none) -> FIT
- C12, C15, C18, C19, C2, C20, C25, C37: MPN (none) -> CL21A106KAYNNNE（华秋 G0022684）; Populate (none) -> FIT
- C16, R21: Populate (none) -> DNP
- C27, C28, C29, C30, C31, C32, C33: MPN (none) -> CL21A475KAQNNNG（华秋 G0936665）; Populate (none) -> FIT
- C34, C35: MPN (none) -> CL10B105KA8NNNC（华秋 G0021698）; Populate (none) -> FIT
- C36: MPN (none) -> 0805B105K250AT（华秋 G4185910）; Populate (none) -> FIT
- R16: MPN (none) -> 0603WAF5231T5E（华秋 G3705144）; Populate (none) -> FIT
- R17: MPN (none) -> RC0603DR-0730K1L（华秋 G4243913）; Populate (none) -> FIT
- R23: MPN (none) -> 0603WAF4703T5E（华秋 G0064373）; Populate (none) -> FIT
- R24: MPN (none) -> RC0603FR-07150KL（华秋 G0072618）; Populate (none) -> FIT
Other:
- note added: "Actuation direction: perpendicular to the PCB surface - the enclosure post presses vertically onto the actuator from the PCB front side."
- note added: "F1-F3 PTC hold current derates with temperature - verify at 25 / 40 / 50 C before claiming 2 A."
- note added: "Power input definition (V1.6): compatible with a 5 V / 2 A source; continuous 2 A at elevated ambient is NOT guaranteed."
- note added: "SW1-SW5 = Omron B3U-1000P (top-actuated tactile switch)"
- note added: "The 90 degree PCB rotation only turns the pads / silkscreen; it does not convert the switch into a side-actuated part."
