File: esp32-board-v1.1/esp32-board-v1.1.kicad_pcb (KiCad board)
At the start: 4 copper layers, 55 x 84 mm, 110 parts, among them J1 USB_C_Receptacle_GCT_USB4105-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, J2 Hirose_FH12-24S-0.5SH_1x24-1M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, J3 microSD_HC_Hirose_DM3AT-SF-PE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, J4 Hirose_DF13-02P-1.25DS_1x02_P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, J5 Hirose_DF13-02P-1.25DS_1x02_P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, Q1 SOT-23, SW1 SW_SPST_B3U-1000P, SW2 SW_SPST_B3U-1000P, SW3 SW_SPST_B3U-1000P, SW4 SW_SPST_B3U-1000P, SW5 SW_SPST_B3U-1000P, U1 ESP32-S3-WROOM-1, U2 Texas_RTW_WQFN-24-1EP_4x4mm_P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, U3 VQFN-16-1EP_3x3mm_P0.5mm_EP1.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, U4 TDFN-8-1EP_2x2mm_P0.5mm_EP0.8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, U5 Texas_X2QFN-12_1.6x1.6mm_P0.4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, U6 SOT-23-6

Commit message: 调整pcb布局
Parts:
- J4, J5: value Hirose_DF13-02P-1.25DS_1x02_P1.25mm_Horizontal -> Molex_PicoBlade_53261-0271_1x02-1MP_P1.25mm_Horizontal; footprint Connector_Hirose:Hirose_DF13-02P-1.25DS_1x02_P1.25mm_Horizontal -> Connector_Molex:Molex_PicoBlade_53261-0271_1x02-1MP_P1.25mm_Horizontal
- moved D3 80.8 mm to (16.0, 82.0)
- moved D5 73.3 mm to (15.9, 78.9)
- moved D2 69.4 mm to (23.8, 74.4)
- moved C6 67.1 mm to (19.4, 71.5)
- moved D4 66.1 mm to (19.5, 74.2)
- moved D1 65.1 mm to (24.0, 71.3)
- moved F1 61.0 mm to (15.1, 75.7)
- moved C7 59.2 mm to (28.5, 69.5)
- moved R8 57.9 mm to (23.2, 68.5)
- moved R11 51.5 mm to (31.2, 67.1)
- moved R12 51.0 mm to (26.5, 65.8)
- moved C8 50.2 mm to (28.5, 63.3)
- moved R36 41.1 mm to (52.0, 55.4)
- moved C38 39.6 mm to (52.5, 76.0)
- moved C37 36.5 mm to (51.1, 63.9)
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
Commit message: 优化pcb布局
Parts:
- removed ? (x4): , MountingHole:MountingHole_2.2mm_M2
- added H1: MountingHole_2.2mm_M2, MountingHole:MountingHole_2.2mm_M2, F.Cu at (3.00, 3.00)
- added H2: MountingHole_2.2mm_M2, MountingHole:MountingHole_2.2mm_M2, F.Cu at (52.0, 3.00)
- added H3: MountingHole_2.2mm_M2, MountingHole:MountingHole_2.2mm_M2, F.Cu at (3.00, 81.0)
- added H4: MountingHole_2.2mm_M2, MountingHole:MountingHole_2.2mm_M2, F.Cu at (52.0, 81.0)
- J2: value Hirose_FH12-24S-0.5SH_1x24-1MP_P0.50mm_Horizontal -> Amphenol_F32Q-1A7x1-11024_1x24-1MP_P0.5mm_Horizontal; footprint Connector_FFC-FPC:Hirose_FH12-24S-0.5SH_1x24-1MP_P0.50mm_Horizontal -> Connector_FFC-FPC:Amphenol_F32Q-1A7x1-11024_1x24-1MP_P0.5mm_Horizontal
- J3: value microSD_HC_Hirose_DM3AT-SF-PEJM5 -> microSD_DM3AT-SF-PEJM5_EPDF; footprint Connector_Card:microSD_HC_Hirose_DM3AT-SF-PEJM5 -> esp32-board-v1.1:microSD_DM3AT-SF-PEJM5_EPDF
- U1: value ESP32-S3-WROOM-1 -> ESP32-S3-WROOM-1_EPDF; footprint RF_Module:ESP32-S3-WROOM-1 -> esp32-board-v1.1:ESP32-S3-WROOM-1_EPDF
- U3: value VQFN-16-1EP_3x3mm_P0.5mm_EP1.45x1.45mm_ThermalVias -> RNM0015A; footprint Package_DFN_QFN:VQFN-16-1EP_3x3mm_P0.5mm_EP1.45x1.45mm_ThermalVias -> esp32-board-v1.1:RNM0015A
- moved R33 51.6 mm to (29.4, 27.5), turned to 0 degrees
- moved R34 46.2 mm to (25.9, 27.5), turned to 0 degrees
- moved C2 30.6 mm to (12.0, 8.28), turned to 180 degrees
- moved R5 29.1 mm to (12.1, 17.9)
- moved C1 29.0 mm to (12.0, 10.7), turned to 180 degrees
- moved R4 28.8 mm to (12.1, 15.4)
- moved R36 28.3 mm to (30.8, 74.3), turned to 90 degrees
- moved C16 27.3 mm to (46.3, 53.3)
- moved C23 26.4 mm to (45.0, 58.2), turned to 90 degrees
- moved R32 26.4 mm to (30.9, 78.0), turned to 90 degrees
- moved C5 25.6 mm to (15.8, 15.4), turned to 180 degrees
- moved R1 24.8 mm to (15.8, 12.9)
- moved R2 24.5 mm to (39.5, 16.8)
- moved C4 24.4 mm to (15.8, 8.03), turned to 180 degrees
- moved C3 24.4 mm to (15.8, 10.5), turned to 180 degrees
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Other:
- board text added: "MOUNTING HOLES:"
- board text added: "NO METAL IN ANTENNA AREA"
- board text added: "NYLON / PLASTIC POST ONLY"
- board text added: "RIGHT_SWITCH_COLUMN"
- board text added: "SW / LOCATING HOLES ONLY"
- board text added: "X 49 - 55 mm"

Commit message: 调整pcb布局
Parts:
- J2: value Amphenol_F32Q-1A7x1-11024_1x24-1MP_P0.5mm_Horizontal -> X05B20U24T; footprint Connector_FFC-FPC:Amphenol_F32Q-1A7x1-11024_1x24-1MP_P0.5mm_Horizontal -> esp32-board-v1.1:X05B20U24T
- L2: value L_Coilcraft_XAL4030-XXX -> L_Sunlord_MWSA0402S; footprint Inductor_SMD:L_Coilcraft_XAL4030-XXX -> Inductor_SMD:L_Sunlord_MWSA0402S
- Q1: value SOT-23 -> SOT-323_SC-70; footprint Package_TO_SOT_SMD:SOT-23 -> Package_TO_SOT_SMD:SOT-323_SC-70
- moved R29 12.7 mm to (12.9, 49.5)
- moved R26 11.2 mm to (40.4, 40.9)
- moved C27 11.1 mm to (20.9, 40.7)
- moved C34 10.4 mm to (11.4, 43.3)
- moved C22 9.05 mm to (33.8, 48.7), turned to 0 degrees
- moved C26 8.58 mm to (13.0, 47.6)
- moved D8 7.60 mm to (15.4, 52.1)
- moved R25 6.79 mm to (29.4, 43.1)
- moved C35 6.27 mm to (17.1, 40.6)
- moved R27 6.26 mm to (43.0, 45.7)
- moved D6 3.31 mm to (20.7, 52.1)
- moved C21 2.50 mm to (42.3, 49.8)
- moved R31 1.81 mm to (19.8, 54.7)
- moved J2 1.73 mm to (3.27, 42.0)
- moved C29 1.50 mm to (22.7, 57.4)
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
Commit message: 更新bom料号
Parts:
- L1: value L_Coilcraft_XAL5030-XXX -> L_Sunlord_MWSA0503S; footprint Inductor_SMD:L_Coilcraft_XAL5030-XXX -> Inductor_SMD:L_Sunlord_MWSA0503S
- L3: value L_Taiyo-Yuden_NR-40xx -> L_Changjiang_FNR4020S; footprint Inductor_SMD:L_Taiyo-Yuden_NR-40xx -> Inductor_SMD:L_Changjiang_FNR4020S

Commit message: 补充料号修正文档
Parts:
- L1: value L_Sunlord_MWSA0503S -> L_Coilcraft_XAL5030-XXX; footprint Inductor_SMD:L_Sunlord_MWSA0503S -> Inductor_SMD:L_Coilcraft_XAL5030-XXX
- L3: value L_Changjiang_FNR4020S -> L_Taiyo-Yuden_NR-40xx; footprint Inductor_SMD:L_Changjiang_FNR4020S -> Inductor_SMD:L_Taiyo-Yuden_NR-40xx

Commit message: 第一轮布线
Routing:
- net SPI_MISO: track 0.00 -> 81.3 mm, vias 0 -> 5
- net KEY3_N: track 0.00 -> 74.3 mm, vias 0 -> 6
- net TF_CD_N: track 0.00 -> 70.7 mm, vias 0 -> 4
- net FG_ALRT_N: track 0.00 -> 67.0 mm, vias 0 -> 2
- net BAT_BUS: track 0.00 -> 65.9 mm, vias 0 -> 2
- net USB_DP_CONN: track 0.00 -> 60.4 mm
- net KEY2_N: track 0.00 -> 54.0 mm, vias 0 -> 3
- net EPD_BUSY: track 0.00 -> 52.3 mm, vias 0 -> 2
- net EPD_PWR_EN: track 0.00 -> 49.1 mm, vias 0 -> 2
- net TF_MOSI: track 0.00 -> 44.6 mm, vias 0 -> 2
- net SPI_SCLK: track 0.00 -> 44.5 mm, vias 0 -> 3
- net EPD_3V3: track 0.00 -> 42.6 mm, vias 0 -> 4
- net KEY1_N: track 0.00 -> 41.4 mm, vias 0 -> 3
- net USB_VBUS_RAW: track 0.00 -> 39.7 mm, vias 0 -> 3
- net SPI_MOSI: track 0.00 -> 38.6 mm, vias 0 -> 3
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- added copper zone on In2.Cu, net GND

Commit message: 第一轮布线优化
Routing:
- net SPI_SCLK: track 44.5 -> 118.0 mm, vias 3 -> 6
- net EPD_VGH: track 0.00 -> 31.9 mm, vias 0 -> 2
- net EPD_DC: track 30.2 -> 60.0 mm
- net EPD_3V3: track 42.6 -> 57.0 mm, vias 4 -> 3
- net SPI_MISO: track 81.3 -> 87.3 mm, vias 5 -> 3
- net EPD_BUSY: track 52.3 -> 56.2 mm
- net FG_ALRT_N: track 67.0 -> 63.2 mm
- net EPD_PWR_EN: track 49.1 -> 52.5 mm
- net KEY3_N: track 74.3 -> 77.1 mm, vias 6 -> 5
- net SPI_MOSI: track 38.6 -> 40.9 mm, vias 3 -> 2
- net TF_CD_N: track 70.7 -> 69.2 mm, vias 4 -> 2
- net EPD_VSH1: track 13.0 -> 14.2 mm
- net KEY2_N: track 54.0 -> 52.8 mm
- net EPD_RST_N: track 33.3 -> 34.4 mm
- net GND: vias 132 -> 135

Commit message: 第二轮布线
Routing:
- net 3V3_MAIN: track 0.00 -> 196.7 mm, vias 0 -> 12
- net SPI_SCLK: track 118.0 -> 45.1 mm, vias 6 -> 3
- net BAT_BUS: track 65.9 -> 0.00 mm, vias 2 -> 0
- net CHG_INT_N: track 0.00 -> 58.4 mm, vias 0 -> 2
- net TF_SCLK: track 0.00 -> 52.7 mm, vias 0 -> 2
- net EPD_3V3: track 57.0 -> 8.68 mm, vias 3 -> 0
- net SYS: track 0.00 -> 41.6 mm, vias 0 -> 2
- net EPD_DC: track 60.0 -> 41.8 mm, vias 2 -> 3
- net TPS_PS_SYNC: track 13.2 -> 0.00 mm, vias 2 -> 0
- net TPS_VSEL: track 9.90 -> 0.00 mm
- net EPD_PWR_EN: track 52.5 -> 43.4 mm
- net EPD_BUSY: track 56.2 -> 47.7 mm, vias 2 -> 3
- net TPS_EN: track 8.20 -> 0.00 mm
- net SPI_MISO: track 87.3 -> 92.0 mm, vias 3 -> 4
- net CHG_ILIM: track 10.7 -> 7.49 mm, vias 0 -> 2
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- added copper zone on F.Cu, net 3V3_MAIN
- added copper zone on F.Cu, net SYS
