File: esp32-board-v1.1/esp32-board-v1.1_power_backbone_checkpoint_20260917.kicad_pcb (KiCad board)
At the start: 4 copper layers, 55 x 84 mm, 110 parts, among them J1 USB_C_Receptacle_GCT_USB4105-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, J2 X05B20U24T, J3 microSD_DM3AT-SF-PEJM5_EPDF, J4 Molex_PicoBlade_53261-0271_1x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, J5 Molex_PicoBlade_53261-0271_1x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, Q1 SOT-323_SC-70, SW1 SW_SPST_B3U-1000P, SW2 SW_SPST_B3U-1000P, SW3 SW_SPST_B3U-1000P, SW4 SW_SPST_B3U-1000P, SW5 SW_SPST_B3U-1000P, U1 ESP32-S3-WROOM-1_EPDF, U2 Texas_RTW_WQFN-24-1EP_4x4mm_P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, U3 RNM0015A, U4 TDFN-8-1EP_2x2mm_P0.5mm_EP0.8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, U5 Texas_X2QFN-12_1.6x1.6mm_P0.4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, U6 SOT-23-6

Commit message: 布线优化
Routing:
- net CHG_CE: track 47.4 -> 0.00 mm, vias 4 -> 0
- net BAT_BUS: track 47.4 -> 0.00 mm, vias 5 -> 0
- net EPD_3V3: track 40.3 -> 14.5 mm, vias 7 -> 0
- net CHG_DSEL: track 17.0 -> 0.00 mm, vias 3 -> 0
- net CHG_REGN: track 7.21 -> 0.00 mm
- net SPI_SCLK: track 43.8 -> 45.1 mm
